File: pic_beeper/pic_beeper.kicad_pcb (KiCad board)
At the start: 2 copper layers, 33 x 26.7 mm, 7 parts, among them J1 Conn_01x06, SW1 SW_SPDT, U1 PIC12F752-IP

Commit message: Code not working
Parts:
- removed BZ1: Buzzer, Buzzer_Beeper:MagneticBuzzer_CUI_CST-931RP-A
- added BZ4: Buzzer, Buzzer_Beeper:Buzzer_12x9.5RM7.6, B.Cu at (6.35, 30.5)
- BT1: footprint lib_fp:BatteryHolder_Q&J-CR2032-BS-6-1 -> lib_fp:BatteryHolder_CR2032_THT; moved to B.Cu
- H1: footprint MountingHole:MountingHole_3.5mm_Pad_Via -> MountingHole:MountingHole_3.5mm_Pad
- J1: footprint lib_fp:PIC_ICSP_Pads_01x06 -> Connector_PinHeader_2.54mm:PinHeader_1x06_P2.54mm_Vertical; moved to B.Cu
- SW1: footprint lib_fp:SW_SPDT_SSAL220100 -> lib_fp:SW_SPDT_Slide_Vertical_THT; moved to B.Cu
- U1: footprint Package_DFN_QFN:DFN-8-1EP_3x3mm_P0.65mm_EP1.55x2.4mm -> Package_DIP:DIP-8_W7.62mm_Socket_LongPads; moved to B.Cu
- moved H1 67.1 mm to (5.08, 5.08)
- moved SW1 63.9 mm to (7.62, 36.8), turned to 180 degrees
- moved BT1 60.8 mm to (14.6, 13.3)
- moved U1 56.7 mm to (16.5, 34.9), turned to 0 degrees
- moved C1 50.7 mm to (16.7, 37.3), turned to 180 degrees
- moved J1 48.4 mm to (29.2, 37.5), turned to 0 degrees
Routing:
- net +BATT: track 15.2 -> 28.0 mm
- net Net-(BT1-Pad1): track 32.8 -> 24.7 mm
- net /BUZZER: track 13.1 -> 20.9 mm
- net -BATT: track 12.0 -> 6.13 mm, vias 4 -> 0
- net /ICSPDAT: track 10.2 -> 6.13 mm, vias 2 -> 0
- net /ICSPCLK: track 7.73 -> 6.13 mm, vias 2 -> 0
- net /VPP: track 15.2 -> 15.9 mm
- added copper zone on F.Cu, net -BATT
- removed copper zone on B.Cu, net -BATT
Other:
- board size 33 x 26.7 mm -> 33 x 40.6 mm
- board text removed: "BEEP BEEP awyea"
- board text removed: "PIC Beeper v1.0 John McNelly"
